Commit message: ankle leveling and pid tuning

File: surena4/src/robot_sim/urdf/surena.xacro (robot description, xacro)
@@ -20,5 +20,5 @@
     </inertial>
     <visual>
-      <origin xyz="0 0 0.951" rpy="0 0 0" />
+      <origin xyz="0 0 0.942" rpy="0 0 0" />
       <geometry>
         <mesh
@@ -32,5 +32,5 @@
     </visual>
     <collision>
-        <origin xyz="0  0 0.951" rpy="1.57 0 0"/>
+        <origin xyz="0  0 0.942" rpy="1.57 0 0"/>
         <geometry>
           <cylinder radius="0.08" length="0.23"/>
@@ -181,12 +181,11 @@
       </material>
     </visual>
-    <collision>
-        <origin xyz="0  0 0" rpy="0 0 0"/>
+    <collision name='RLeg_Foot_Link_collision'>
+        <origin xyz=".045  0 -.09" rpy="0 0 0"/>
         <geometry>
-        <mesh
-          filename="package://robot_sim/meshes/Foot-Right.STL" />
+           <box size="0.26 0.16 0.02"/>
         </geometry>
-      </collision>
-  </link>
+     </collision>
+</link>
 <link name="LLeg_HipY_Link">
 <inertial>
@@ -332,44 +331,73 @@
       </material>
     </visual>
+    <collision  name='LLeg_Foot_Link_collision'>
+    <origin xyz=".045  0 -.09" rpy="0 0 0"/>
+        <geometry>
+          <box size="0.26 0.16 0.02"/>
+        </geometry>
+    </collision>
+  </link>
+<gazebo reference="LLeg_Foot_Link">
+        <mu1>3</mu1>
+        <mu2>3</mu2>
+        <kp>2000000.0</kp>
+</gazebo>
+<gazebo reference="RLeg_Foot_Link">
+        <mu1>3</mu1>
+         <mu2>3</mu2>
+        <kp>2000000.0</kp>
+</gazebo>
+<link name="WAIST_LINK1">
+<inertial>
+      <origin
+        xyz="0 -0 0.0 "
+        rpy="0 0 0" />
+      <mass
+        value="2.50321784932644" />
+      <inertia
+        ixx="0.0344409751913919"
+        ixy="0.000203000704156372"
+        ixz="-0.000402443503216186"
+        iyy="0.0459468264001583"
+        iyz="-0.00410422593827533"
+        izz="0.0404358469485904" />
+    </inertial>
     <collision>
         <origin xyz="0  0 0" rpy="0 0 0"/>
         <geometry>
         <mesh
-          filename="package://robot_sim/meshes/Foot-Left.STL" />
+          filename="package://robot_sim/meshes/tORSO.STL" />
         </geometry>
       </collision>
-      <surface>
-            <friction>
-              <ode>
-                <mu>1</mu>
-                <mu2>1</mu2>
-                <fdir1>0 0 1</fdir1>
-                <slip1>0.0</slip1>
-                <slip2>0.0</slip2>
-              </ode>
-            </friction>
-            <contact>
-                 <ode>
-                    <min_depth>5</min_depth>
-                     <kp>1e8</kp>
-                 </ode>
-            </contact>
-      </surface>
-  </link>
-<link name="WAIST_LINK1">
-<inertial>
-      <origin
-        xyz="0 -0 0.0 "
-        rpy="0 0 0" />
-      <mass
-        value="2.50321784932644" />
-      <inertia
-        ixx="0.0344409751913919"
-        ixy="0.000203000704156372"
-        ixz="-0.000402443503216186"
-        iyy="0.0459468264001583"
-        iyz="-0.00410422593827533"
-        izz="0.0404358469485904" />
-    </inertial>
+  </link>
+<link name="WAIST_LINK2">
+<inertial>
+      <origin
+        xyz="0 -0 0.0 "
+        rpy="0 0 0" />
+      <mass
+        value="2.50321784932644" />
+      <inertia
+        ixx="0.0344409751913919"
+        ixy="0.000203000704156372"
+        ixz="-0.000402443503216186"
+        iyy="0.0459468264001583"
+        iyz="-0.00410422593827533"
+        izz="0.0404358469485904" />
+    </inertial>
+    <visual>
+      <origin
+        xyz="0 0 0"
+        rpy="0 0 0" />
+      <geometry>
+        <mesh
+          filename="package://robot_sim/meshes/tORSO.STL" />
+      </geometry>
+      <material
+        name="">
+        <color
+          rgba="0.792156862745098 0.819607843137255 0.933333333333333 1" />
+      </material>
+    </visual>
     <collision>
         <origin xyz="0  0 0" rpy="0 0 0"/>
@@ -380,20 +408,52 @@
       </collision>
   </link>
-<link name="WAIST_LINK2">
-<inertial>
-      <origin
-        xyz="0 -0 0.0 "
-        rpy="0 0 0" />
-      <mass
-        value="2.50321784932644" />
-      <inertia
-        ixx="0.0344409751913919"
-        ixy="0.000203000704156372"
-        ixz="-0.000402443503216186"
-        iyy="0.0459468264001583"
-        iyz="-0.00410422593827533"
-        izz="0.0404358469485904" />
-    </inertial>
-    <visual>
+<link name="RARM_LINK1">
+<inertial>
+      <origin
+        xyz="0 -0 0.0 "
+        rpy="0 0 0" />
+      <mass
+        value="2.50321784932644" />
+      <inertia
+        ixx="0.0344409751913919"
+        ixy="0.000203000704156372"
+        ixz="-0.000402443503216186"
+        iyy="0.0459468264001583"
+        iyz="-0.00410422593827533"
+        izz="0.0404358469485904" />
+    </inertial>
+  </link>
+<link name="RARM_LINK2">
+<inertial>
+      <origin
+        xyz="0 -0 0.0 "
+        rpy="0 0 0" />
+      <mass
+        value="2.50321784932644" />
+      <inertia
+        ixx="0.0344409751913919"
+        ixy="0.000203000704156372"
+        ixz="-0.000402443503216186"
+        iyy="0.0459468264001583"
+        iyz="-0.00410422593827533"
+        izz="0.0404358469485904" />
+    </inertial>
+  </link>
+<link name="RARM_LINK3">
+<inertial>
+      <origin
+        xyz="0 -0 0.0 "
+        rpy="0 0 0" />
+      <mass
+        value="2.50321784932644" />
+      <inertia
+        ixx="0.0344409751913919"
+        ixy="0.000203000704156372"
+        ixz="-0.000402443503216186"
+        iyy="0.0459468264001583"
+        iyz="-0.00410422593827533"
+        izz="0.0404358469485904" />
+    </inertial>
+<visual>
       <origin
         xyz="0 0 0"
@@ -401,5 +461,5 @@
       <geometry>
         <mesh
-          filename="package://robot_sim/meshes/tORSO.STL" />
+          filename="package://robot_sim/meshes/Upper-arm-right.STL" />
       </geometry>
       <material
@@ -413,56 +473,24 @@
         <geometry>
         <mesh
-          filename="package://robot_sim/meshes/tORSO.STL" />
+          filename="package://robot_sim/meshes/Upper-arm-right.STL" />
         </geometry>
       </collision>
   </link>
-<link name="RARM_LINK1">
-<inertial>
-      <origin
-        xyz="0 -0 0.0 "
-        rpy="0 0 0" />
-      <mass
-        value="2.50321784932644" />
-      <inertia
-        ixx="0.0344409751913919"
-        ixy="0.000203000704156372"
-        ixz="-0.000402443503216186"
-        iyy="0.0459468264001583"
-        iyz="-0.00410422593827533"
-        izz="0.0404358469485904" />
-    </inertial>
-  </link>
-<link name="RARM_LINK2">
-<inertial>
-      <origin
-        xyz="0 -0 0.0 "
-        rpy="0 0 0" />
-      <mass
-        value="2.50321784932644" />
-      <inertia
-        ixx="0.0344409751913919"
-        ixy="0.000203000704156372"
-        ixz="-0.000402443503216186"
-        iyy="0.0459468264001583"
-        iyz="-0.00410422593827533"
-        izz="0.0404358469485904" />
-    </inertial>
-  </link>
-<link name="RARM_LINK3">
-<inertial>
-      <origin
-        xyz="0 -0 0.0 "
-        rpy="0 0 0" />
-      <mass
-        value="2.50321784932644" />
-      <inertia
-        ixx="0.0344409751913919"
-        ixy="0.000203000704156372"
-        ixz="-0.000402443503216186"
-        iyy="0.0459468264001583"
-        iyz="-0.00410422593827533"
-        izz="0.0404358469485904" />
-    </inertial>
-<visual>
+<link name="RARM_LINK4">
+<inertial>
+      <origin
+        xyz="0 -0 0.0 "
+        rpy="0 0 0" />
+      <mass
+        value="2.50321784932644" />
+      <inertia
+        ixx="0.0344409751913919"
+        ixy="0.000203000704156372"
+        ixz="-0.000402443503216186"
+        iyy="0.0459468264001583"
+        iyz="-0.00410422593827533"
+        izz="0.0404358469485904" />
+    </inertial>
+    <visual>
       <origin
         xyz="0 0 0"
@@ -470,5 +498,67 @@
       <geometry>
         <mesh
-          filename="package://robot_sim/meshes/Upper-arm-right.STL" />
+          filename="package://robot_sim/meshes/fore-arm-right.STL" />
+      </geometry>
+      <material
+        name="">
+        <color
+          rgba="0.792156862745098 0.819607843137255 0.933333333333333 1" />
+      </material>
+    </visual>
+  </link>
+<link name="RARM_LINK5">
+<inertial>
+      <origin
+        xyz="0 -0 0.0 "
+        rpy="0 0 0" />
+      <mass
+        value="2.50321784932644" />
+      <inertia
+        ixx="0.0344409751913919"
+        ixy="0.000203000704156372"
+        ixz="-0.000402443503216186"
+        iyy="0.0459468264001583"
+        iyz="-0.00410422593827533"
+        izz="0.0404358469485904" />
+    </inertial>
+  </link>
+<link name="RARM_LINK6">
+<inertial>
+      <origin
+        xyz="0 -0 0.0 "
+        rpy="0 0 0" />
+      <mass
+        value="2.50321784932644" />
+      <inertia
+        ixx="0.0344409751913919"
+        ixy="0.000203000704156372"
+        ixz="-0.000402443503216186"
+        iyy="0.0459468264001583"
+        iyz="-0.00410422593827533"
+        izz="0.0404358469485904" />
+    </inertial>
+  </link>
+<link name="RARM_LINK7">
+<inertial>
+      <origin
+        xyz="0 -0 0.0 "
+        rpy="0 0 0" />
+      <mass
+        value="2.50321784932644" />
+      <inertia
+        ixx="0.0344409751913919"
+        ixy="0.000203000704156372"
+        ixz="-0.000402443503216186"
+        iyy="0.0459468264001583"
+        iyz="-0.00410422593827533"
+        izz="0.0404358469485904" />
+    </inertial>
+    <visual>
+      <origin
+        xyz="0 0 0"
+        rpy="0 0 0" />
+      <geometry>
+        <mesh
+          filename="package://robot_sim/meshes/Hand-Right.STL" />
       </geometry>
       <material
@@ -482,24 +572,56 @@
         <geometry>
         <mesh
-          filename="package://robot_sim/meshes/Upper-arm-right.STL" />
+          filename="package://robot_sim/meshes/Hand-Right.STL" />
         </geometry>
       </collision>
   </link>
-<link name="RARM_LINK4">
-<inertial>
-      <origin
-        xyz="0 -0 0.0 "
-        rpy="0 0 0" />
-      <mass
-        value="2.50321784932644" />
-      <inertia
-        ixx="0.0344409751913919"
-        ixy="0.000203000704156372"
-        ixz="-0.000402443503216186"
-        iyy="0.0459468264001583"
-        iyz="-0.00410422593827533"
-        izz="0.0404358469485904" />
-    </inertial>
-    <visual>
+<link name="LARM_LINK1">
+<inertial>
+      <origin
+        xyz="0 -0 0.0 "
+        rpy="0 0 0" />
+      <mass
+        value="2.50321784932644" />
+      <inertia
+        ixx="0.0344409751913919"
+        ixy="0.000203000704156372"
+        ixz="-0.000402443503216186"
+        iyy="0.0459468264001583"
+        iyz="-0.00410422593827533"
+        izz="0.0404358469485904" />
+    </inertial>
+  </link>
+<link name="LARM_LINK2">
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