Commit message: hand codes added and gazebo model update

File: surena4/src/robot_sim/urdf/surena.xacro (robot description, xacro)
@@ -7,15 +7,15 @@
 <inertial>
       <origin
-        xyz="0 0.0 0.0 "
-        rpy="0 0 0" />
-      <mass
-        value="30" />
-      <inertia
-        ixx="0.0344409751913919"
-        ixy="0.000203000704156372"
-        ixz="-0.000402443503216186"
-        iyy="0.0459468264001583"
-        iyz="-0.00410422593827533"
-        izz="0.0404358469485904" />
+        xyz="-0.0517 0 0.9727 "
+        rpy="0 0 0" />
+      <mass
+        value="2.3" />
+      <inertia
+        ixx="0.001365"
+        ixy="0.000068"
+        ixz="-0.000361"
+        iyy="0.006717"
+        iyz="-0.000089"
+        izz="0.001752" />
     </inertial>
     <visual>
@@ -32,5 +32,5 @@
     </visual>
     <collision>
-        <origin xyz="0  0 0.942" rpy="1.57 0 0"/>
+        <origin xyz="0  0 0.942" rpy="1.57 0 0.0"/>
         <geometry>
           <cylinder radius="0.08" length="0.23"/>
@@ -40,26 +40,26 @@
 <link name="RLeg_HipY_Link">
 <inertial>
-      <origin xyz="0 -0 0 " rpy="0 0 0" />
-      <mass value="2.50321784932644" />
-      <inertia
-        ixx="0.0344409751913919"
-        ixy="0.000203000704156372"
-        ixz="-0.000402443503216186"
-        iyy="0.0459468264001583"
-        iyz="-0.00410422593827533"
-        izz="0.0404358469485904" />
+      <origin xyz="-0.067 0 -0.059 " rpy="0 0 0" />
+      <mass value="1.29" />
+      <inertia
+        ixx="0.005106"
+        ixy="0.000029"
+        ixz="0.003622"
+        iyy="0.011031"
+        iyz="0.000013"
+        izz="0.007143" />
     </inertial>
   </link>
 <link name="RLeg_Hip_Uni_Link">
 <inertial>
-      <origin xyz="0 -0 0 " rpy="0 0 0" />
-      <mass value="5" />
-      <inertia
-        ixx="0.0344409751913919"
-        ixy="0.000203000704156372"
-        ixz="-0.000402443503216186"
-        iyy="0.0459468264001583"
-        iyz="-0.00410422593827533"
-        izz="0.0404358469485904" />
+      <origin xyz="-0.003 -0.002 -0.0004 " rpy="0 0 0" />
+      <mass value="1.15" />
+      <inertia
+        ixx="0.001754"
+        ixy="-0.000017"
+        ixz="0.000034"
+        iyy="0.001753"
+        iyz="0.000002"
+        izz="0.025712" />
     </inertial>
   </link>
@@ -67,15 +67,15 @@
 <inertial>
       <origin
-        xyz="0 -0 0 "
-        rpy="0 0 0" />
-      <mass
-        value="2.50321784932644" />
-      <inertia
-        ixx="0.0344409751913919"
-        ixy="0.000203000704156372"
-        ixz="-0.000402443503216186"
-        iyy="0.0459468264001583"
-        iyz="-0.00410422593827533"
-        izz="0.0404358469485904" />
+        xyz="0.002 0.001 -0.19 "
+        rpy="0 0 0" />
+      <mass
+        value="2.08" />
+      <inertia
+        ixx="0.031121"
+        ixy="-0.00004"
+        ixz="-0.000024"
+        iyy="0.029521"
+        iyz="0.000317"
+        izz="0.006842" />
     </inertial>
     <visual>
@@ -103,15 +103,15 @@
 <inertial>
       <origin
-        xyz="0 -0 0.0 "
-        rpy="0 0 0" />
-      <mass
-        value="2.50321784932644" />
-      <inertia
-        ixx="0.0344409751913919"
-        ixy="0.000203000704156372"
-        ixz="-0.000402443503216186"
-        iyy="0.0459468264001583"
-        iyz="-0.00410422593827533"
-        izz="0.0404358469485904" />
+        xyz="0.0013 0.0014 -0.09 "
+        rpy="0 0 0" />
+      <mass
+        value="4.85" />
+      <inertia
+        ixx="0.059549"
+        ixy="0.000020"
+        ixz="-0.000220"
+        iyy="0.055950"
+        iyz="0.001301"
+        izz="0.009826" />
     </inertial>
     <visual>
@@ -139,15 +139,15 @@
 <inertial>
       <origin
-        xyz="0 -0 0.0 "
-        rpy="0 0 0" />
-      <mass
-        value="2.50321784932644" />
-      <inertia
-        ixx="0.0344409751913919"
-        ixy="0.000203000704156372"
-        ixz="-0.000402443503216186"
-        iyy="0.0459468264001583"
-        iyz="-0.00410422593827533"
-        izz="0.0404358469485904" />
+        xyz="-0.029 -0.0017 0.057 "
+        rpy="0 0 0" />
+      <mass
+        value="2.49" />
+      <inertia
+      ixx="0.028025"
+      ixy="-0.000028"
+      ixz="-0.004505"
+      iyy="0.029547"
+      iyz="-0.000618"
+      izz="0.006102" />
     </inertial>
   </link>
@@ -155,15 +155,15 @@
 <inertial>
       <origin
-        xyz="0 -0 0.0 "
-        rpy="0 0 0" />
-      <mass
-        value="2.50321784932644" />
-      <inertia
-        ixx="0.0344409751913919"
-        ixy="0.000203000704156372"
-        ixz="-0.000402443503216186"
-        iyy="0.0459468264001583"
-        iyz="-0.00410422593827533"
-        izz="0.0404358469485904" />
+        xyz="0.0055 0.0012 -0.072 "
+        rpy="0 0 0" />
+      <mass
+        value="1.48" />
+      <inertia
+      ixx="0.001702"
+      ixy="0.000013"
+      ixz="-0.000187"
+      iyy="0.003158"
+      iyz="-0.000031"
+      izz="0.003625"/>
     </inertial>
     <visual>
@@ -190,26 +190,26 @@
 <link name="LLeg_HipY_Link">
 <inertial>
-      <origin xyz="0 -0 0 " rpy="0 0 0" />
-      <mass value="2.50321784932644" />
-      <inertia
-        ixx="0.0344409751913919"
-        ixy="0.000203000704156372"
-        ixz="-0.000402443503216186"
-        iyy="0.0459468264001583"
-        iyz="-0.00410422593827533"
-        izz="0.0404358469485904" />
+      <origin xyz="-0.067 0 -0.059 " rpy="0 0 0" />
+      <mass value="1.29" />
+      <inertia
+      ixx="0.005106"
+      ixy="-0.000029"
+      ixz="0.003622"
+      iyy="0.011031"
+      iyz="-0.000013"
+      izz="0.007143" />
     </inertial>
   </link>
 <link name="LLeg_Hip_Uni_Link">
 <inertial>
-      <origin xyz="0 -0 0 " rpy="0 0 0" />
-      <mass value="2.50321784932644" />
-      <inertia
-        ixx="0.0344409751913919"
-        ixy="0.000203000704156372"
-        ixz="-0.000402443503216186"
-        iyy="0.0459468264001583"
-        iyz="-0.00410422593827533"
-        izz="0.0404358469485904" />
+      <origin xyz="-0.003 0.002 -0.0004 " rpy="0 0 0" />
+      <mass value="1.15" />
+      <inertia
+      ixx="0.001754"
+      ixy="0.000017"
+      ixz="0.000034"
+      iyy="0.001753"
+      iyz="-0.000002"
+      izz="0.025712" />
     </inertial>
   </link>
@@ -217,15 +217,15 @@
 <inertial>
       <origin
-        xyz="0 -0 0 "
-        rpy="0 0 0" />
-      <mass
-        value="2.50321784932644" />
-      <inertia
-        ixx="0.0344409751913919"
-        ixy="0.000203000704156372"
-        ixz="-0.000402443503216186"
-        iyy="0.0459468264001583"
-        iyz="-0.00410422593827533"
-        izz="0.0404358469485904" />
+        xyz="0.002 -0.001 -0.19 "
+        rpy="0 0 0" />
+      <mass
+        value="2.08" />
+      <inertia
+      ixx="0.031121"
+      ixy="0.00004"
+      ixz="-0.000024"
+      iyy="0.029521"
+      iyz="-0.000317"
+      izz="0.006842" />
     </inertial>
     <visual>
@@ -236,4 +236,40 @@
         <mesh
           filename="package://robot_sim/meshes/Thigh-Left.STL" />
+      </geometry>
+      <material
+        name="">
+        <color
+          rgba="0.792156862745098 0.819607843137255 0.933333333333333 1" />
+      </material>
+    </visual>
+    <collision>
+        <origin xyz="0 0 -0.18" rpy="0 0 0"/>
+        <geometry>
+          <cylinder radius="0.04" length="0.35"/>
+        </geometry>
+      </collision>
+  </link>
+<link name="LLeg_Hip_Shank_Link">
+<inertial>
+      <origin
+        xyz="0.0013 -0.0014 -0.09  "
+        rpy="0 0 0" />
+      <mass
+        value="4.85" />
+      <inertia
+      ixx="0.059549"
+      ixy="-0.000020"
+      ixz="-0.000220"
+      iyy="0.055950"
+      iyz="-0.001301"
+      izz="0.009826" />
+    </inertial>
+    <visual>
+      <origin
+        xyz="0 0 0"
+        rpy="0 0 0" />
+      <geometry>
+        <mesh
+          filename="package://robot_sim/meshes/Shank-Left.STL" />
       </geometry>
       <material
@@ -250,54 +286,18 @@
       </collision>
   </link>
-<link name="LLeg_Hip_Shank_Link">
-<inertial>
-      <origin
-        xyz="0 -0 0.0 "
-        rpy="0 0 0" />
-      <mass
-        value="2.50321784932644" />
-      <inertia
-        ixx="0.0344409751913919"
-        ixy="0.000203000704156372"
-        ixz="-0.000402443503216186"
-        iyy="0.0459468264001583"
-        iyz="-0.00410422593827533"
-        izz="0.0404358469485904" />
-    </inertial>
-    <visual>
-      <origin
-        xyz="0 0 0"
-        rpy="0 0 0" />
-      <geometry>
-        <mesh
-          filename="package://robot_sim/meshes/Shank-Left.STL" />
-      </geometry>
-      <material
-        name="">
-        <color
-          rgba="0.792156862745098 0.819607843137255 0.933333333333333 1" />
-      </material>
-    </visual>
-    <collision>
-        <origin xyz="0  0 -0.18" rpy="0 0 0"/>
-        <geometry>
-          <cylinder radius="0.04" length="0.35"/>
-        </geometry>
-      </collision>
-  </link>
 <link name="LLeg_Ankle_Uni_Link">
 <inertial>
       <origin
-        xyz="0 -0 0.0 "
-        rpy="0 0 0" />
-      <mass
-        value="2.50321784932644" />
-      <inertia
-        ixx="0.0344409751913919"
-        ixy="0.000203000704156372"
-        ixz="-0.000402443503216186"
-        iyy="0.0459468264001583"
-        iyz="-0.00410422593827533"
-        izz="0.0404358469485904" />
+        xyz="-0.029 0.0017 0.057  "
+        rpy="0 0 0" />
+      <mass
+        value="2.49" />
+      <inertia
+        ixx="0.028025"
+        ixy="0.000028"
+        ixz="-0.004505"
+        iyy="0.029547"
+        iyz="0.000618"
+        izz="0.006102" />
     </inertial>
   </link>
@@ -305,15 +305,15 @@
 <inertial>
       <origin
-        xyz="0 -0 0.0 "
-        rpy="0 0 0" />
-      <mass
-        value="2.50321784932644" />
-      <inertia
-        ixx="0.0344409751913919"
-        ixy="0.000203000704156372"
-        ixz="-0.000402443503216186"
-        iyy="0.0459468264001583"
-        iyz="-0.00410422593827533"
-        izz="0.0404358469485904" />
+        xyz="0.0055 -0.0012 -0.072 "
+        rpy="0 0 0" />
+      <mass
+        value="1.48" />
+      <inertia
+        ixx="0.001702"
+        ixy="-0.000013"
+        ixz="-0.000187"
+        iyy="0.003158"
+        iyz="0.000031"
+        izz="0.003625" />
     </inertial>
     <visual>
@@ -351,294 +351,287 @@
 <inertial>
       <origin
-        xyz="0 -0 0.0 "
-        rpy="0 0 0" />
-      <mass
-        value="2.50321784932644" />
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
File: surena4/src/robot_sim/urdf/surena2.xacro (robot description, xacro)
@@ -1,4 +1,4 @@
 <?xml version='1.0'?>
-<robot name="surena" xmlns:xacro="http://www.ros.org/wiki/xacro">
+<robot name="rrbot" xmlns:xacro="http://www.ros.org/wiki/xacro">
 <!--  <xacro:include filename="$(find robot_sim)/urdf/surena.gazebo" />
   <xacro:include filename="$(find robot_sim)/urdf/materials.xacro" />
@@ -10,5 +10,5 @@
         rpy="0 0 0" />
       <mass
-        value="2.50321784932644" />
+        value="3" />
       <inertia
         ixx="0.0344409751913919"
@@ -20,5 +20,5 @@
     </inertial>
     <visual>
-      <origin xyz="0 0 0.951" rpy="0 0 0" />
+      <origin xyz="0 0 0.942" rpy="0 0 0" />
       <geometry>
         <mesh
@@ -32,5 +32,5 @@
     </visual>
     <collision>
-        <origin xyz="0  0 0.951" rpy="1.57 0 0"/>
+        <origin xyz="0  0 0.942" rpy="1.57 0 0"/>
         <geometry>
           <cylinder radius="0.08" length="0.23"/>
@@ -54,5 +54,5 @@
 <inertial>
       <origin xyz="0 -0 0 " rpy="0 0 0" />
-      <mass value="2.50321784932644" />
+      <mass value="5" />
       <inertia
         ixx="0.0344409751913919"
@@ -181,12 +181,11 @@
       </material>
     </visual>
-    <collision>
-        <origin xyz="0  0 0" rpy="0 0 0"/>
+    <collision name='RLeg_Foot_Link_collision'>
+        <origin xyz=".045  0 -.09" rpy="0 0 0"/>
         <geometry>
-        <mesh
-          filename="package://robot_sim/meshes/Foot-Right.STL" />
+           <box size="0.26 0.16 0.02"/>
         </geometry>
-      </collision>
-  </link>
+     </collision>
+</link>
 <link name="LLeg_HipY_Link">
 <inertial>
@@ -332,25 +331,431 @@
       </material>
     </visual>
+    <collision  name='LLeg_Foot_Link_collision'>
+    <origin xyz=".045  0 -.09" rpy="0 0 0"/>
+        <geometry>
+          <box size="0.26 0.16 0.02"/>
+        </geometry>
+    </collision>
+  </link>
+<gazebo reference="LLeg_Foot_Link">
+        <mu1>3</mu1>
+        <mu2>3</mu2>
+        <kp>2000000.0</kp>
+</gazebo>
+<gazebo reference="RLeg_Foot_Link">
+        <mu1>3</mu1>
+         <mu2>3</mu2>
+        <kp>2000000.0</kp>
+</gazebo>
+<link name="WAIST_LINK1">
+<inertial>
+      <origin
+        xyz="0 -0 0.0 "
+        rpy="0 0 0" />
+      <mass
+        value="2.50321784932644" />
+      <inertia
+        ixx="0.0344409751913919"
+        ixy="0.000203000704156372"
+        ixz="-0.000402443503216186"
+        iyy="0.0459468264001583"
+        iyz="-0.00410422593827533"
+        izz="0.0404358469485904" />
+    </inertial>
     <collision>
         <origin xyz="0  0 0" rpy="0 0 0"/>
         <geometry>
         <mesh
-          filename="package://robot_sim/meshes/Foot-Left.STL" />
+          filename="package://robot_sim/meshes/tORSO.STL" />
         </geometry>
       </collision>
   </link>
+<link name="WAIST_LINK2">
+<inertial>
+      <origin
+        xyz="0 -0 0.0 "
+        rpy="0 0 0" />
+      <mass
+        value="2.50321784932644" />
+      <inertia
+        ixx="0.0344409751913919"
+        ixy="0.000203000704156372"
+        ixz="-0.000402443503216186"
+        iyy="0.0459468264001583"
+        iyz="-0.00410422593827533"
+        izz="0.0404358469485904" />
+    </inertial>
+    <visual>
+      <origin
+        xyz="0 0 0"
+        rpy="0 0 0" />
+      <geometry>
+        <mesh
+          filename="package://robot_sim/meshes/tORSO.STL" />
+      </geometry>
+      <material
+        name="">
+        <color
+          rgba="0.792156862745098 0.819607843137255 0.933333333333333 1" />
+      </material>
+    </visual>
+    <collision>
+        <origin xyz="0  0 0" rpy="0 0 0"/>
+        <geometry>
+        <mesh
+          filename="package://robot_sim/meshes/tORSO.STL" />
+        </geometry>
+      </collision>
+  </link>
+<link name="RARM_LINK1">
+<inertial>
+      <origin
+        xyz="0 -0 0.0 "
+        rpy="0 0 0" />
+      <mass
+        value="2.50321784932644" />
+      <inertia
+        ixx="0.0344409751913919"
+        ixy="0.000203000704156372"
+        ixz="-0.000402443503216186"
+        iyy="0.0459468264001583"
+        iyz="-0.00410422593827533"
+        izz="0.0404358469485904" />
+    </inertial>
+  </link>
+<link name="RARM_LINK2">
+<inertial>
+      <origin
+        xyz="0 -0 0.0 "
+        rpy="0 0 0" />
+      <mass
+        value="2.50321784932644" />
+      <inertia
+        ixx="0.0344409751913919"
+        ixy="0.000203000704156372"
+        ixz="-0.000402443503216186"
+        iyy="0.0459468264001583"
+        iyz="-0.00410422593827533"
+        izz="0.0404358469485904" />
+    </inertial>
+  </link>
+<link name="RARM_LINK3">
+<inertial>
+      <origin
+        xyz="0 -0 0.0 "
+        rpy="0 0 0" />
+      <mass
+        value="2.50321784932644" />
+      <inertia
+        ixx="0.0344409751913919"
+        ixy="0.000203000704156372"
+        ixz="-0.000402443503216186"
+        iyy="0.0459468264001583"
+        iyz="-0.00410422593827533"
+        izz="0.0404358469485904" />
+    </inertial>
+<visual>
+      <origin
+        xyz="0 0 0"
+        rpy="0 0 0" />
+      <geometry>
+        <mesh
+          filename="package://robot_sim/meshes/Upper-arm-right.STL" />
+      </geometry>
+      <material
+        name="">
+        <color
+          rgba="0.792156862745098 0.819607843137255 0.933333333333333 1" />
+      </material>
+    </visual>
+    <collision>
+        <origin xyz="0  0 0" rpy="0 0 0"/>
+        <geometry>
+        <mesh
+          filename="package://robot_sim/meshes/Upper-arm-right.STL" />
+        </geometry>
+      </collision>
+  </link>
+<link name="RARM_LINK4">
+<inertial>
+      <origin
+        xyz="0 -0 0.0 "
+        rpy="0 0 0" />
+      <mass
+        value="2.50321784932644" />
+      <inertia
+        ixx="0.0344409751913919"
+        ixy="0.000203000704156372"
+        ixz="-0.000402443503216186"
+        iyy="0.0459468264001583"
+        iyz="-0.00410422593827533"
+        izz="0.0404358469485904" />
+    </inertial>
+    <visual>
+      <origin
+        xyz="0 0 0"
+        rpy="0 0 0" />
+      <geometry>
+        <mesh
+          filename="package://robot_sim/meshes/fore-arm-right.STL" />
+      </geometry>
+      <material
+        name="">
+        <color
+          rgba="0.792156862745098 0.819607843137255 0.933333333333333 1" />
+      </material>
+    </visual>
+  </link>
+<link name="RARM_LINK5">
+<inertial>
+      <origin
+        xyz="0 -0 0.0 "
+        rpy="0 0 0" />
+      <mass
+        value="2.50321784932644" />
+      <inertia
+        ixx="0.0344409751913919"
+        ixy="0.000203000704156372"
+        ixz="-0.000402443503216186"
+        iyy="0.0459468264001583"
+        iyz="-0.00410422593827533"
+        izz="0.0404358469485904" />
+    </inertial>
+  </link>
+<link name="RARM_LINK6">
+<inertial>
+      <origin
+        xyz="0 -0 0.0 "
+        rpy="0 0 0" />
+      <mass
+        value="2.50321784932644" />
+      <inertia
+        ixx="0.0344409751913919"
+        ixy="0.000203000704156372"
+        ixz="-0.000402443503216186"
+        iyy="0.0459468264001583"
+        iyz="-0.00410422593827533"
+        izz="0.0404358469485904" />
+    </inertial>
+  </link>
+<link name="RARM_LINK7">
+<inertial>
+      <origin
+        xyz="0 -0 0.0 "
+        rpy="0 0 0" />
+      <mass
+        value="2.50321784932644" />
+      <inertia
+        ixx="0.0344409751913919"
+        ixy="0.000203000704156372"
+        ixz="-0.000402443503216186"
+        iyy="0.0459468264001583"
+        iyz="-0.00410422593827533"
+        izz="0.0404358469485904" />
+    </inertial>
+    <visual>
+      <origin
+        xyz="0 0 0"
+        rpy="0 0 0" />
+      <geometry>
+        <mesh
+          filename="package://robot_sim/meshes/Hand-Right.STL" />
+      </geometry>
+      <material
+        name="">
+        <color
+          rgba="0.792156862745098 0.819607843137255 0.933333333333333 1" />
+      </material>
+    </visual>
+    <collision>
+        <origin xyz="0  0 0" rpy="0 0 0"/>
+        <geometry>
+        <mesh
+          filename="package://robot_sim/meshes/Hand-Right.STL" />
+        </geometry>
+      </collision>
+  </link>
+<link name="LARM_LINK1">
+<inertial>
+      <origin
+        xyz="0 -0 0.0 "
+        rpy="0 0 0" />
+      <mass
+        value="2.50321784932644" />
+      <inertia
+        ixx="0.0344409751913919"
+        ixy="0.000203000704156372"
+        ixz="-0.000402443503216186"
+        iyy="0.0459468264001583"
+        iyz="-0.00410422593827533"
+        izz="0.0404358469485904" />
+    </inertial>
+  </link>
+<link name="LARM_LINK2">
+<inertial>
+      <origin
+        xyz="0 -0 0.0 "
+        rpy="0 0 0" />
+      <mass
+        value="2.50321784932644" />
+      <inertia
+        ixx="0.0344409751913919"
+        ixy="0.000203000704156372"
+        ixz="-0.000402443503216186"
+        iyy="0.0459468264001583"
+        iyz="-0.00410422593827533"
+        izz="0.0404358469485904" />
+    </inertial>
+  </link>
+<link name="LARM_LINK3">
+<inertial>
+      <origin
+        xyz="0 -0 0.0 "
+        rpy="0 0 0" />
+      <mass
+        value="2.50321784932644" />
+      <inertia
+        ixx="0.0344409751913919"
+        ixy="0.000203000704156372"
+        ixz="-0.000402443503216186"
+        iyy="0.0459468264001583"
+        iyz="-0.00410422593827533"
+        izz="0.0404358469485904" />
+    </inertial>
+  <visual>
+      <origin
+        xyz="0 0 0"
+        rpy="0 0 0" />
+      <geometry>
+        <mesh
+          filename="package://robot_sim/meshes/Upper-arm-Left.STL" />
+      </geometry>
+      <material
+        name="">
+        <color
+          rgba="0.792156862745098 0.819607843137255 0.933333333333333 1" />
+      </material>
+    </visual>
+    <collision>
+        <origin xyz="0  0 0" rpy="0 0 0"/>
+        <geometry>
+        <mesh
+          filename="package://robot_sim/meshes/Upper-arm-Left.STL" />
+        </geometry>
+      </collision>
+  </link>
+<link name="LARM_LINK4">
+<inertial>
+      <origin
+        xyz="0 -0 0.0 "
+        rpy="0 0 0" />
+      <mass
+        value="2.50321784932644" />
+      <inertia
+        ixx="0.0344409751913919"
+        ixy="0.000203000704156372"
+        ixz="-0.000402443503216186"
+        iyy="0.0459468264001583"
+        iyz="-0.00410422593827533"
+        izz="0.0404358469485904" />
+    </inertial>
+    <visual>
+      <origin
+        xyz="0 0 0"
+        rpy="0 0 0" />
+      <geometry>
+        <mesh
+          filename="package://robot_sim/meshes/fore-arm-Left.STL" />
+      </geometry>
+      <material
+        name="">
+        <color
+          rgba="0.792156862745098 0.819607843137255 0.933333333333333 1" />
+      </material>
+    </visual>
+  </link>
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