Commit message: start surena-eth node

File: surena4/src/robot_sim/urdf/surena.xacro (robot description, xacro)
@@ -4,5 +4,5 @@
   <xacro:include filename="$(find robot_sim)/urdf/materials.xacro" />
   <xacro:include filename="$(find robot_sim)/urdf/macros.xacro" />-->
-<link name="pelvis">
+<link name="base_link">
 <inertial>
       <origin
@@ -746,12 +746,12 @@
 <joint name="RLeg_HipY_J1" type="continuous">
    <origin xyz="0 -0.115 0.942 " rpy="0 0 0"/>
-   <parent link="pelvis"/>
+   <parent link="base_link"/>
    <child link="RLeg_HipY_Link"/>
    <axis xyz="0 0 1"/>
     <limit effort="300.0" lower="-1000" upper="-1000" velocity="0.5"/>
  </joint>
-<transmission name="J1t">
-   <type>transmission_interface/SimpleTransmission</type>
-   <actuator name="motor1">
+<transmission name="RLeg_HipY_J1">
+   <type>transmission_interface/SimpleTransmission</type>
+   <actuator name="RLeg_HipY_J1">
      <mechanicalReduction>1</mechanicalReduction>
    </actuator>
@@ -767,5 +767,5 @@
     <limit effort="300.0" lower="-1000" upper="-1000" velocity="0.5"/>
   </joint>
-<transmission name="J2t">
+<transmission name="RLeg_HipR_J2">
    <type>transmission_interface/SimpleTransmission</type>
    <actuator name="motor2">
@@ -783,5 +783,5 @@
       <limit effort="300.0" lower="-1000" upper="-1000" velocity="0.5"/>
    </joint>
-<transmission name="J3t">
+<transmission name="RLeg_HipP_J3">
    <type>transmission_interface/SimpleTransmission</type>
    <actuator name="motor3">
@@ -799,5 +799,5 @@
      <limit effort="300.0" lower="-1000" upper="-1000" velocity="0.5"/>
   </joint>
-<transmission name="J4t">
+<transmission name="RLeg_KneeP_J4">
    <type>transmission_interface/SimpleTransmission</type>
    <actuator name="motor4">
@@ -815,5 +815,5 @@
     <limit effort="300.0" lower="-1000" upper="-1000" velocity="0.5"/>
  </joint>
-<transmission name="J5t">
+<transmission name="RLeg_AnkleP_J5">
    <type>transmission_interface/SimpleTransmission</type>
    <actuator name="motor5">
@@ -831,5 +831,5 @@
     <limit effort="300.0" lower="-1000" upper="-1000" velocity="0.5"/>
  </joint>
-<transmission name="J6t">
+<transmission name="RLeg_AnkleR_J6">
    <type>transmission_interface/SimpleTransmission</type>
    <actuator name="motor6">
@@ -842,10 +842,10 @@
 <joint name="LLeg_HipY_J1" type="continuous">
    <origin xyz="0 +0.115 0.942 " rpy="0 0 0"/>
-   <parent link="pelvis"/>
+   <parent link="base_link"/>
    <child link="LLeg_HipY_Link"/>
    <axis xyz="0 0 1"/>
     <limit effort="300.0" lower="-1000" upper="-1000" velocity="0.5"/>
  </joint>
-<transmission name="J7t">
+<transmission name="LLeg_HipY_J1">
    <type>transmission_interface/SimpleTransmission</type>
    <actuator name="motor7">
@@ -863,5 +863,5 @@
      <limit effort="300.0" lower="-1000" upper="-1000" velocity="0.5"/>
   </joint>
-<transmission name="J8t">
+<transmission name="LLeg_HipR_J2">
    <type>transmission_interface/SimpleTransmission</type>
    <actuator name="motor8">
@@ -879,5 +879,5 @@
       <limit effort="300.0" lower="-1000" upper="-1000" velocity="0.5"/>
    </joint>
-<transmission name="J9t">
+<transmission name="LLeg_HipP_J3">
    <type>transmission_interface/SimpleTransmission</type>
    <actuator name="motor9">
@@ -895,5 +895,5 @@
      <limit effort="300.0" lower="-1000" upper="-1000" velocity="0.5"/>
   </joint>
-<transmission name="J10t">
+<transmission name="LLeg_KneeP_J4">
    <type>transmission_interface/SimpleTransmission</type>
    <actuator name="motor10">
@@ -911,5 +911,5 @@
     <limit effort="300.0" lower="-1000" upper="-1000" velocity="0.5"/>
  </joint>
-<transmission name="J11t">
+<transmission name="LLeg_AnkleP_J5">
    <type>transmission_interface/SimpleTransmission</type>
    <actuator name="motor11">
@@ -927,5 +927,5 @@
     <limit effort="300.0" lower="-1000" upper="-1000" velocity="0.5"/>
  </joint>
-<transmission name="J12t">
+<transmission name="LLeg_AnkleR_J6">
    <type>transmission_interface/SimpleTransmission</type>
    <actuator name="motor12">
@@ -938,10 +938,10 @@
 <joint name="Waist_Y_J1" type="continuous">
    <origin xyz="0 0.0 1.071" rpy="0 0 0"/>
-   <parent link="pelvis"/>
+   <parent link="base_link"/>
    <child link="WAIST_LINK1"/>
    <axis xyz="0 0 1"/>
     <limit effort="300.0" lower="-1000" upper="-1000" velocity="0.5"/>
  </joint>
-<transmission name="J13t">
+<transmission name="Waist_Y_J1">
    <type>transmission_interface/SimpleTransmission</type>
    <actuator name="motor13">
@@ -959,5 +959,5 @@
     <limit effort="300.0" lower="-1000" upper="-1000" velocity="0.5"/>
  </joint>
-<transmission name="J14t">
+<transmission name="Waist_Y_J2">
    <type>transmission_interface/SimpleTransmission</type>
    <actuator name="motor14">
@@ -975,5 +975,5 @@
     <limit effort="300.0" lower="-1000" upper="-1000" velocity="0.5"/>
  </joint>
-<transmission name="J15t">
+<transmission name="RArm_ShoulderP_J1">
    <type>transmission_interface/SimpleTransmission</type>
    <actuator name="motor15">
@@ -991,5 +991,5 @@
     <limit effort="300.0" lower="-1000" upper="-1000" velocity="0.5"/>
  </joint>
-<transmission name="J16t">
+<transmission name="RArm_ShoulderR_J2">
    <type>transmission_interface/SimpleTransmission</type>
    <actuator name="motor16">
@@ -1007,5 +1007,5 @@
     <limit effort="300.0" lower="-1000" upper="-1000" velocity="0.5"/>
  </joint>
-<transmission name="J17t">
+<transmission name="RArm_ShoulderY_J3">
    <type>transmission_interface/SimpleTransmission</type>
    <actuator name="motor17">
@@ -1023,5 +1023,5 @@
     <limit effort="300.0" lower="-1000" upper="-1000" velocity="0.5"/>
  </joint>
-<transmission name="J18t">
+<transmission name="RArm_ElbowP_J4">
    <type>transmission_interface/SimpleTransmission</type>
    <actuator name="motor18">
@@ -1039,5 +1039,5 @@
     <limit effort="300.0" lower="-1000" upper="-1000" velocity="0.5"/>
  </joint>
-<transmission name="J19t">
+<transmission name="RArm_WristY_J5">
    <type>transmission_interface/SimpleTransmission</type>
    <actuator name="motor19">
@@ -1055,5 +1055,5 @@
     <limit effort="300.0" lower="-1000" upper="-1000" velocity="0.5"/>
  </joint>
-<transmission name="J20t">
+<transmission name="RArm_WristR_J6">
    <type>transmission_interface/SimpleTransmission</type>
    <actuator name="motor20">
@@ -1071,5 +1071,5 @@
     <limit effort="300.0" lower="-1000" upper="-1000" velocity="0.5"/>
  </joint>
-<transmission name="J21t">
+<transmission name="RArm_WristP_J7">
    <type>transmission_interface/SimpleTransmission</type>
    <actuator name="motor21">
@@ -1087,5 +1087,5 @@
     <limit effort="300.0" lower="-1000" upper="-1000" velocity="0.5"/>
  </joint>
-<transmission name="J22t">
+<transmission name="LArm_ShoulderP_J1">
    <type>transmission_interface/SimpleTransmission</type>
    <actuator name="motor22">
@@ -1103,5 +1103,5 @@
     <limit effort="300.0" lower="-1000" upper="-1000" velocity="0.5"/>
  </joint>
-<transmission name="J23t">
+<transmission name="LArm_ShoulderR_J2">
    <type>transmission_interface/SimpleTransmission</type>
    <actuator name="motor23">
@@ -1119,5 +1119,5 @@
     <limit effort="300.0" lower="-1000" upper="-1000" velocity="0.5"/>
  </joint>
-<transmission name="J24t">
+<transmission name="LArm_ShoulderY_J3">
    <type>transmission_interface/SimpleTransmission</type>
    <actuator name="motor24">
@@ -1135,5 +1135,5 @@
     <limit effort="300.0" lower="-1000" upper="-1000" velocity="0.5"/>
  </joint>
-<transmission name="J25t">
+<transmission name="LArm_ElbowP_J4">
    <type>transmission_interface/SimpleTransmission</type>
    <actuator name="motor25">
@@ -1151,5 +1151,5 @@
     <limit effort="300.0" lower="-1000" upper="-1000" velocity="0.5"/>
  </joint>
-<transmission name="J26t">
+<transmission name="LArm_WristY_J5">
    <type>transmission_interface/SimpleTransmission</type>
    <actuator name="motor26">
@@ -1167,5 +1167,5 @@
     <limit effort="300.0" lower="-1000" upper="-1000" velocity="0.5"/>
  </joint>
-<transmission name="J27t">
+<transmission name="LArm_WristR_J6">
    <type>transmission_interface/SimpleTransmission</type>
    <actuator name="motor27">
@@ -1183,5 +1183,5 @@
     <limit effort="300.0" lower="-1000" upper="-1000" velocity="0.5"/>
  </joint>
-<transmission name="J28t">
+<transmission name="LArm_WristP_J7">
    <type>transmission_interface/SimpleTransmission</type>
    <actuator name="motor28">

File: surena4/src/robot_sim/urdf/surena2.xacro (robot description, xacro)
@@ -1,8 +1,8 @@
 <?xml version='1.0'?>
-<robot name="surena" xmlns:xacro="http://www.ros.org/wiki/xacro">
+<robot name="rrbot" xmlns:xacro="http://www.ros.org/wiki/xacro">
 <!--  <xacro:include filename="$(find robot_sim)/urdf/surena.gazebo" />
   <xacro:include filename="$(find robot_sim)/urdf/materials.xacro" />
   <xacro:include filename="$(find robot_sim)/urdf/macros.xacro" />-->
-<link name="pelvis">
+<link name="base_link">
 <inertial>
       <origin
@@ -10,5 +10,5 @@
         rpy="0 0 0" />
       <mass
-        value="2.50321784932644" />
+        value="30" />
       <inertia
         ixx="0.0344409751913919"
@@ -20,5 +20,5 @@
     </inertial>
     <visual>
-      <origin xyz="0 0 0.951" rpy="0 0 0" />
+      <origin xyz="0 0 0.942" rpy="0 0 0" />
       <geometry>
         <mesh
@@ -32,5 +32,5 @@
     </visual>
     <collision>
-        <origin xyz="0  0 0.951" rpy="1.57 0 0"/>
+        <origin xyz="0  0 0.942" rpy="1.57 0 0"/>
         <geometry>
           <cylinder radius="0.08" length="0.23"/>
@@ -54,5 +54,5 @@
 <inertial>
       <origin xyz="0 -0 0 " rpy="0 0 0" />
-      <mass value="2.50321784932644" />
+      <mass value="5" />
       <inertia
         ixx="0.0344409751913919"
@@ -181,12 +181,11 @@
       </material>
     </visual>
-    <collision>
-        <origin xyz="0  0 0" rpy="0 0 0"/>
+    <collision name='RLeg_Foot_Link_collision'>
+        <origin xyz=".045  0 -.09" rpy="0 0 0"/>
         <geometry>
-        <mesh
-          filename="package://robot_sim/meshes/Foot-Right.STL" />
+           <box size="0.26 0.16 0.02"/>
         </geometry>
-      </collision>
-  </link>
+     </collision>
+</link>
 <link name="LLeg_HipY_Link">
 <inertial>
@@ -332,25 +331,431 @@
       </material>
     </visual>
+    <collision  name='LLeg_Foot_Link_collision'>
+    <origin xyz=".045  0 -.09" rpy="0 0 0"/>
+        <geometry>
+          <box size="0.26 0.16 0.02"/>
+        </geometry>
+    </collision>
+  </link>
+<gazebo reference="LLeg_Foot_Link">
+        <mu1>3</mu1>
+        <mu2>3</mu2>
+        <kp>2000000.0</kp>
+</gazebo>
+<gazebo reference="RLeg_Foot_Link">
+        <mu1>3</mu1>
+         <mu2>3</mu2>
+        <kp>2000000.0</kp>
+</gazebo>
+<link name="WAIST_LINK1">
+<inertial>
+      <origin
+        xyz="0 -0 0.0 "
+        rpy="0 0 0" />
+      <mass
+        value="2.50321784932644" />
+      <inertia
+        ixx="0.0344409751913919"
+        ixy="0.000203000704156372"
+        ixz="-0.000402443503216186"
+        iyy="0.0459468264001583"
+        iyz="-0.00410422593827533"
+        izz="0.0404358469485904" />
+    </inertial>
     <collision>
         <origin xyz="0  0 0" rpy="0 0 0"/>
         <geometry>
         <mesh
-          filename="package://robot_sim/meshes/Foot-Left.STL" />
+          filename="package://robot_sim/meshes/tORSO.STL" />
         </geometry>
       </collision>
   </link>
+<link name="WAIST_LINK2">
+<inertial>
+      <origin
+        xyz="0 -0 0.0 "
+        rpy="0 0 0" />
+      <mass
+        value="2.50321784932644" />
+      <inertia
+        ixx="0.0344409751913919"
+        ixy="0.000203000704156372"
+        ixz="-0.000402443503216186"
+        iyy="0.0459468264001583"
+        iyz="-0.00410422593827533"
+        izz="0.0404358469485904" />
+    </inertial>
+    <visual>
+      <origin
+        xyz="0 0 0"
+        rpy="0 0 0" />
+      <geometry>
+        <mesh
+          filename="package://robot_sim/meshes/tORSO.STL" />
+      </geometry>
+      <material
+        name="">
+        <color
+          rgba="0.792156862745098 0.819607843137255 0.933333333333333 1" />
+      </material>
+    </visual>
+    <collision>
+        <origin xyz="0  0 0" rpy="0 0 0"/>
+        <geometry>
+        <mesh
+          filename="package://robot_sim/meshes/tORSO.STL" />
+        </geometry>
+      </collision>
+  </link>
+<link name="RARM_LINK1">
+<inertial>
+      <origin
+        xyz="0 -0 0.0 "
+        rpy="0 0 0" />
+      <mass
+        value="2.50321784932644" />
+      <inertia
+        ixx="0.0344409751913919"
+        ixy="0.000203000704156372"
+        ixz="-0.000402443503216186"
+        iyy="0.0459468264001583"
+        iyz="-0.00410422593827533"
+        izz="0.0404358469485904" />
+    </inertial>
+  </link>
+<link name="RARM_LINK2">
+<inertial>
+      <origin
+        xyz="0 -0 0.0 "
+        rpy="0 0 0" />
+      <mass
+        value="2.50321784932644" />
+      <inertia
+        ixx="0.0344409751913919"
+        ixy="0.000203000704156372"
+        ixz="-0.000402443503216186"
+        iyy="0.0459468264001583"
+        iyz="-0.00410422593827533"
+        izz="0.0404358469485904" />
+    </inertial>
+  </link>
+<link name="RARM_LINK3">
+<inertial>
+      <origin
+        xyz="0 -0 0.0 "
+        rpy="0 0 0" />
+      <mass
+        value="2.50321784932644" />
+      <inertia
+        ixx="0.0344409751913919"
+        ixy="0.000203000704156372"
+        ixz="-0.000402443503216186"
+        iyy="0.0459468264001583"
+        iyz="-0.00410422593827533"
+        izz="0.0404358469485904" />
+    </inertial>
+<visual>
+      <origin
+        xyz="0 0 0"
+        rpy="0 0 0" />
+      <geometry>
+        <mesh
+          filename="package://robot_sim/meshes/Upper-arm-right.STL" />
+      </geometry>
+      <material
+        name="">
+        <color
+          rgba="0.792156862745098 0.819607843137255 0.933333333333333 1" />
+      </material>
+    </visual>
+    <collision>
+        <origin xyz="0  0 0" rpy="0 0 0"/>
+        <geometry>
+        <mesh
+          filename="package://robot_sim/meshes/Upper-arm-right.STL" />
+        </geometry>
+      </collision>
+  </link>
+<link name="RARM_LINK4">
+<inertial>
+      <origin
+        xyz="0 -0 0.0 "
+        rpy="0 0 0" />
+      <mass
+        value="2.50321784932644" />
+      <inertia
+        ixx="0.0344409751913919"
+        ixy="0.000203000704156372"
+        ixz="-0.000402443503216186"
+        iyy="0.0459468264001583"
+        iyz="-0.00410422593827533"
+        izz="0.0404358469485904" />
+    </inertial>
+    <visual>
+      <origin
+        xyz="0 0 0"
+        rpy="0 0 0" />
+      <geometry>
+        <mesh
+          filename="package://robot_sim/meshes/fore-arm-right.STL" />
+      </geometry>
+      <material
+        name="">
+        <color
+          rgba="0.792156862745098 0.819607843137255 0.933333333333333 1" />
+      </material>
+    </visual>
+  </link>
+<link name="RARM_LINK5">
+<inertial>
+      <origin
+        xyz="0 -0 0.0 "
+        rpy="0 0 0" />
+      <mass
+        value="2.50321784932644" />
+      <inertia
+        ixx="0.0344409751913919"
+        ixy="0.000203000704156372"
+        ixz="-0.000402443503216186"
+        iyy="0.0459468264001583"
+        iyz="-0.00410422593827533"
+        izz="0.0404358469485904" />
+    </inertial>
+  </link>
+<link name="RARM_LINK6">
+<inertial>
+      <origin
+        xyz="0 -0 0.0 "
+        rpy="0 0 0" />
+      <mass
+        value="2.50321784932644" />
+      <inertia
+        ixx="0.0344409751913919"
+        ixy="0.000203000704156372"
+        ixz="-0.000402443503216186"
+        iyy="0.0459468264001583"
+        iyz="-0.00410422593827533"
+        izz="0.0404358469485904" />
+    </inertial>
+  </link>
+<link name="RARM_LINK7">
+<inertial>
+      <origin
+        xyz="0 -0 0.0 "
+        rpy="0 0 0" />
+      <mass
+        value="2.50321784932644" />
+      <inertia
+        ixx="0.0344409751913919"
+        ixy="0.000203000704156372"
+        ixz="-0.000402443503216186"
+        iyy="0.0459468264001583"
+        iyz="-0.00410422593827533"
+        izz="0.0404358469485904" />
+    </inertial>
+    <visual>
+      <origin
+        xyz="0 0 0"
+        rpy="0 0 0" />
+      <geometry>
+        <mesh
+          filename="package://robot_sim/meshes/Hand-Right.STL" />
+      </geometry>
+      <material
+        name="">
+        <color
+          rgba="0.792156862745098 0.819607843137255 0.933333333333333 1" />
+      </material>
+    </visual>
+    <collision>
+        <origin xyz="0  0 0" rpy="0 0 0"/>
+        <geometry>
+        <mesh
+          filename="package://robot_sim/meshes/Hand-Right.STL" />
+        </geometry>
+      </collision>
+  </link>
+<link name="LARM_LINK1">
+<inertial>
+      <origin
+        xyz="0 -0 0.0 "
+        rpy="0 0 0" />
+      <mass
+        value="2.50321784932644" />
+      <inertia
+        ixx="0.0344409751913919"
+        ixy="0.000203000704156372"
+        ixz="-0.000402443503216186"
+        iyy="0.0459468264001583"
+        iyz="-0.00410422593827533"
+        izz="0.0404358469485904" />
+    </inertial>
+  </link>
+<link name="LARM_LINK2">
+<inertial>
+      <origin
+        xyz="0 -0 0.0 "
+        rpy="0 0 0" />
+      <mass
+        value="2.50321784932644" />
+      <inertia
+        ixx="0.0344409751913919"
+        ixy="0.000203000704156372"
+        ixz="-0.000402443503216186"
+        iyy="0.0459468264001583"
+        iyz="-0.00410422593827533"
+        izz="0.0404358469485904" />
+    </inertial>
+  </link>
+<link name="LARM_LINK3">
+<inertial>
+      <origin
+        xyz="0 -0 0.0 "
+        rpy="0 0 0" />
+      <mass
+        value="2.50321784932644" />
+      <inertia
+        ixx="0.0344409751913919"
+        ixy="0.000203000704156372"
+        ixz="-0.000402443503216186"
+        iyy="0.0459468264001583"
+        iyz="-0.00410422593827533"
+        izz="0.0404358469485904" />
+    </inertial>
+  <visual>
+      <origin
+        xyz="0 0 0"
+        rpy="0 0 0" />
+      <geometry>
+        <mesh
+          filename="package://robot_sim/meshes/Upper-arm-Left.STL" />
+      </geometry>
+      <material
+        name="">
+        <color
+          rgba="0.792156862745098 0.819607843137255 0.933333333333333 1" />
+      </material>
+    </visual>
+    <collision>
+        <origin xyz="0  0 0" rpy="0 0 0"/>
+        <geometry>
+        <mesh
+          filename="package://robot_sim/meshes/Upper-arm-Left.STL" />
+        </geometry>
+      </collision>
+  </link>
+<link name="LARM_LINK4">
+<inertial>
+      <origin
+        xyz="0 -0 0.0 "
+        rpy="0 0 0" />
+      <mass
+        value="2.50321784932644" />
+      <inertia
+        ixx="0.0344409751913919"
+        ixy="0.000203000704156372"
+        ixz="-0.000402443503216186"
+        iyy="0.0459468264001583"
+        iyz="-0.00410422593827533"
+        izz="0.0404358469485904" />
+    </inertial>
+    <visual>
+      <origin
+        xyz="0 0 0"
+        rpy="0 0 0" />
+      <geometry>
+        <mesh
+          filename="package://robot_sim/meshes/fore-arm-Left.STL" />
+      </geometry>
+      <material
+        name="">
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
Commit message: params ok and hands added to surena-eth

File: surena4/src/robot_sim/urdf/surena.xacro (robot description, xacro)
@@ -182,5 +182,5 @@
     </visual>
     <collision name='RLeg_Foot_Link_collision'>
-        <origin xyz=".045  0 -.09" rpy="0 0 0"/>
+        <origin xyz=".045  0 -.1" rpy="0 0 0"/>
         <geometry>
            <box size="0.26 0.16 0.02"/>
@@ -332,5 +332,5 @@
     </visual>
     <collision  name='LLeg_Foot_Link_collision'>
-    <origin xyz=".045  0 -.09" rpy="0 0 0"/>
+    <origin xyz=".045  0 -.1" rpy="0 0 0"/>
         <geometry>
           <box size="0.26 0.16 0.02"/>
@@ -962,5 +962,5 @@
  </transmission>
 <joint name="RArm_ShoulderP_J1" type="continuous">
-   <origin xyz="0  -0.207 0.2694" rpy="-0.174533 0 0"/>
+   <origin xyz="0  -0.239 0.2694" rpy="-0.174533 0 0"/>
    <parent link="WAIST_LINK2"/>
    <child link="RARM_LINK1"/>
@@ -1074,5 +1074,5 @@
  </transmission>
 <joint name="LArm_ShoulderP_J1" type="continuous">
-   <origin xyz="0 0.207 0.2694" rpy="0.174533 0 0"/>
+   <origin xyz="0 0.239 0.2694" rpy="0.174533 0 0"/>
    <parent link="WAIST_LINK2"/>
    <child link="LARM_LINK1"/>
